File: devboard.kicad_pcb (KiCad board)
At the start: 2 copper layers, 0 parts

Commit message: layout is my biggest opp </3
Parts:
- added C1: 1uF, Capacitor_SMD:C_0402_1005Metric, F.Cu at (178.7, 87.1)
- added C10: 1uF, Capacitor_SMD:C_0402_1005Metric, F.Cu at (160.0, 76.6)
- added C11: 0.1uF, Capacitor_SMD:C_0402_1005Metric, F.Cu at (164.9, 68.0)
- added C12: 0.1uF, Capacitor_SMD:C_0402_1005Metric, F.Cu at (159.9, 74.6)
- added C13: 10uF, Capacitor_SMD:C_0603_1608Metric, F.Cu at (163.4, 64.0)
- added C14: 10uF, Capacitor_SMD:C_0603_1608Metric, F.Cu at (166.2, 60.2)
- added C15: 33pF, Capacitor_SMD:C_0402_1005Metric, F.Cu at (163.2, 80.9)
- added C16: 33pF, Capacitor_SMD:C_0402_1005Metric, F.Cu at (157.6, 80.9)
- added C17: 0.1uF, Capacitor_SMD:C_0402_1005Metric, F.Cu at (164.9, 70.4)
- added C2: 0.1uF, Capacitor_SMD:C_0402_1005Metric, F.Cu at (162.1, 74.5)
- added C3: 0.1uF, Capacitor_SMD:C_0402_1005Metric, F.Cu at (154.9, 70.6)
- added C4: 0.1uF, Capacitor_SMD:C_0402_1005Metric, F.Cu at (160.5, 95.0)
- added C5: 0.1uF, Capacitor_SMD:C_0402_1005Metric, F.Cu at (157.8, 74.6)
- added C6: 0.1uF, Capacitor_SMD:C_0402_1005Metric, F.Cu at (155.9, 62.5)
- added C7: 0.1uF, Capacitor_SMD:C_0402_1005Metric, F.Cu at (162.8, 85.0)
- added C8: 0.1uF, Capacitor_SMD:C_0402_1005Metric, F.Cu at (158.4, 84.9)
- added C9: 0.1uF, Capacitor_SMD:C_0402_1005Metric, F.Cu at (160.7, 85.0)
- added J1: USB_C_Receptacle_USB2.0_14P, Connector_USB:USB_C_Receptacle_HRO_TYPE-C-31-M-12, F.Cu at (160.7, 53.3)
- added J2: Conn_01x03, Connector_PinHeader_2.54mm:PinHeader_1x03_P2.54mm_Vertical, F.Cu at (158.0, 100.1)
- added J3: Conn_01x20, Connector_PinHeader_2.54mm:PinHeader_1x20_P2.54mm_Vertical, F.Cu at (151.6, 52.3)
- added J4: Conn_01x20, Connector_PinHeader_2.54mm:PinHeader_1x20_P2.54mm_Vertical, F.Cu at (169.7, 52.3)
- added R1: 5.1K, Resistor_SMD:R_0402_1005Metric, F.Cu at (182.3, 74.5)
- added R2: 5.1K, Resistor_SMD:R_0402_1005Metric, F.Cu at (182.3, 76.5)
- added R3: 27, Resistor_SMD:R_0402_1005Metric, F.Cu at (182.3, 78.5)
- added R4: 27, Resistor_SMD:R_0402_1005Metric, F.Cu at (182.3, 80.5)
- added R5: 1K, Resistor_SMD:R_0402_1005Metric, F.Cu at (182.3, 82.5)
- added R6: 10K, Resistor_SMD:R_0402_1005Metric, F.Cu at (175.0, 92.4)
- added R7: 1K, Resistor_SMD:R_0402_1005Metric, F.Cu at (154.8, 67.0)
- added SW1: SW_Push, Button_Switch_SMD:SW_Push_SPST_NO_Alps_SKRK, F.Cu at (165.4, 76.0)
- added U1: RP2040, Package_DFN_QFN:QFN-56-1EP_7x7mm_P0.4mm_EP3.2x3.2mm, F.Cu at (160.1, 69.5)
- added U2: NCP1117-3.3_SOT223, Package_TO_SOT_SMD:SOT-223-3_TabPin2, F.Cu at (160.7, 90.0)
- added U3: W25Q16JVZPIQ TR, Package_SON:Winbond_USON-8-1EP_3x2mm_P0.5mm_EP0.2x1.6mm, F.Cu at (158.2, 62.8)
- added U4: MCP1700x-330xxTT, Package_TO_SOT_SMD:SOT-23, F.Cu at (163.4, 60.5)
- added Y1: 12 MHz, Crystal:Crystal_SMD_3225-4Pin_3.2x2.5mm, F.Cu at (160.4, 80.8)
Other:
- board outline added: 21 x 51 mm
- board text removed: "lol"

Commit message: some routing (help me)
Parts:
- moved R6 35.5 mm to (156.0, 62.4), turned to 180 degrees
- moved C4 27.9 mm to (155.4, 67.5), turned to 180 degrees
- moved R4 26.6 mm to (160.9, 64.6), turned to -90 degrees
- moved R3 24.4 mm to (161.9, 65.1), turned to 90 degrees
- moved C1 22.9 mm to (165.7, 68.2)
- moved R7 11.9 mm to (157.7, 78.5)
- moved C10 11.8 mm to (162.9, 65.2), turned to 90 degrees
- moved C7 10.8 mm to (165.4, 74.5), turned to 90 degrees
- moved C5 10.4 mm to (164.0, 66.2), turned to 90 degrees
- moved C17 9.85 mm to (160.9, 61.4), turned to -90 degrees
- moved C3 8.80 mm to (158.1, 62.4)
- moved C2 8.46 mm to (165.6, 66.8), turned to 25 degrees
- moved C9 8.33 mm to (162.1, 76.8), turned to 90 degrees
- moved C11 7.00 mm to (159.9, 63.0)
- moved C13 6.26 mm to (158.8, 59.7)
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Routing:
- net +3V3: track 0.00 -> 19.5 mm, vias 0 -> 2
- net USB_D+: track 0.00 -> 11.6 mm
- net USB_D-: track 0.00 -> 11.5 mm
- net QSPI_SS: track 0.00 -> 8.74 mm
- net QSPI_SD2: track 0.00 -> 7.83 mm
- net QSPI_SD1: track 0.00 -> 6.82 mm
- net QSPI_SD3: track 0.00 -> 4.40 mm
- net +1V1: track 0.00 -> 4.10 mm
- net QSPI_SCLK: track 0.00 -> 3.67 mm
- net QSPI_SD0: track 0.00 -> 2.96 mm
- net Net-(U1-USB_DP): track 0.00 -> 2.61 mm
- net Net-(U1-USB_DM): track 0.00 -> 2.09 mm

Commit message: routing done. i am crashing out over drc lol
Parts:
- moved J4 48.4 mm to (169.7, 100.6), turned to 180 degrees
- moved R2 29.6 mm to (158.3, 59.2), turned to 180 degrees
- moved R5 22.8 mm to (160.3, 76.4), turned to 180 degrees
- moved R1 21.0 mm to (164.3, 63.6)
- moved C8 17.8 mm to (166.6, 71.5), turned to 0 degrees
- moved C14 11.6 mm to (155.6, 59.8), turned to 180 degrees
- moved C7 11.3 mm to (154.3, 72.8), turned to 180 degrees
- moved C13 9.02 mm to (166.0, 65.2)
- moved C15 8.88 mm to (155.9, 78.9), turned to 90 degrees
- moved R7 6.07 mm to (154.7, 83.8)
- moved C16 4.51 mm to (161.2, 79.8), turned to -90 degrees
- moved Y1 3.92 mm to (158.6, 79.3), turned to 180 degrees
- moved C12 3.16 mm to (163.0, 77.4), turned to -90 degrees
- moved U4 1.85 mm to (165.8, 60.6)
- moved C9 1.34 mm to (161.3, 77.9), turned to -90 degrees
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Connections:
- J4 pad 1: GPIO15 -> GPIO16
Routing:
- net VBUS: track 0.00 -> 71.4 mm, vias 0 -> 2
- net RUN: track 0.00 -> 42.9 mm, vias 0 -> 1
- net +3V3: track 19.5 -> 59.0 mm, vias 2 -> 3
- net GPIO15: track 0.00 -> 31.0 mm, vias 0 -> 1
- net GPIO16: track 0.00 -> 30.2 mm
- net SWCLK: track 0.00 -> 29.7 mm, vias 0 -> 1
- net SWD: track 0.00 -> 29.7 mm, vias 0 -> 1
- net GPIO14: track 0.00 -> 28.5 mm
- net GPIO17: track 0.00 -> 28.1 mm
- net GPIO13: track 0.00 -> 23.4 mm, vias 0 -> 1
- net GPIO12: track 0.00 -> 23.3 mm
- net GPIO18: track 0.00 -> 22.3 mm, vias 0 -> 1
- net GPIO19: track 0.00 -> 20.3 mm, vias 0 -> 1
- net GPIO0: track 0.00 -> 19.9 mm, vias 0 -> 1
- net GPIO1: track 0.00 -> 18.6 mm, vias 0 -> 1
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- added copper zone on B.Cu, net GND
- added copper zone on F.Cu, net GND
Other:
- board size 21 x 51 mm -> 21.9 x 51.5 mm
