File: _autosave-devboard.kicad_pcb (KiCad board)
At the start: 2 copper layers, 20.9 x 51.2 mm, 38 parts, among them J1 USB_C_Receptacle_USB2.0_14P, J2 Conn_01x03, J3 Conn_01x20, J4 Conn_01x20, SW1 SW_Push, U1 RP2040, U2 NCP1117-3.3_SOT223, U3 W25Q16JVZPIQ TR, U4 MCP1700x-330xxTT, Y1 12 MHz

Commit message: done! added finishing touches
Parts:
- removed the G*** at (175.1, 65.0)
- removed the G*** at (169.3, 119.4)
- moved G*** 2.70 mm to (158.6, 77.6)
